Commit message: Center mass fixed

File: urdf/bot5.xacro (robot description, xacro)
@@ -6,5 +6,5 @@
 <link name="base_link">
   <inertial>
-    <origin xyz="0.02411436877412949 -0.0002108801413928273 0.15999684267558398" rpy="0 0 0"/>
+    <origin xyz="-0.1758856312258705 -0.0002108801413928246 0.15999684267558398" rpy="0 0 0"/>
     <mass value="8.70709040372319"/>
     <inertia ixx="0.077475" iyy="0.211713" izz="0.269158" ixy="0.000108" iyz="-1.7e-05" ixz="-0.006764"/>
@@ -26,10 +26,10 @@
 <link name="left_wheel_1">
   <inertial>
-    <origin xyz="4.860168806375409e-05 0.03873115898033333 -4.449218771185315e-14" rpy="0 0 0"/>
+    <origin xyz="0.20004860168806374 0.03873115898033333 -4.449218771185315e-14" rpy="0 0 0"/>
     <mass value="2.1920210431083533"/>
     <inertia ixx="0.008637" iyy="0.016397" izz="0.008644" ixy="-3e-06" iyz="-0.0" ixz="-0.0"/>
   </inertial>
   <visual>
-    <origin xyz="-0.194069 -0.149879 -0.125" rpy="0 0 0"/>
+    <origin xyz="0.205931 -0.149879 -0.125" rpy="0 0 0"/>
     <geometry>
       <mesh filename="package://bot5_description/meshes/left_wheel_1.stl" scale="0.001 0.001 0.001"/>
@@ -38,5 +38,5 @@
   </visual>
   <collision>
-    <origin xyz="-0.194069 -0.149879 -0.125" rpy="0 0 0"/>
+    <origin xyz="0.205931 -0.149879 -0.125" rpy="0 0 0"/>
     <geometry>
       <mesh filename="package://bot5_description/meshes/left_wheel_1.stl" scale="0.001 0.001 0.001"/>
@@ -46,10 +46,10 @@
 <link name="right_wheel_1">
   <inertial>
-    <origin xyz="4.860168807085952e-05 -0.03873122504117252 -4.4103609653234344e-14" rpy="0 0 0"/>
+    <origin xyz="0.20004860168807084 -0.03873122504117252 -4.4103609653234344e-14" rpy="0 0 0"/>
     <mass value="2.1920210431083507"/>
-    <inertia ixx="0.008637" iyy="0.016397" izz="0.008644" ixy="3e-06" iyz="-0.0" ixz="0.0"/>
-  </inertial>
-  <visual>
-    <origin xyz="-0.194069 0.150121 -0.125" rpy="0 0 0"/>
+    <inertia ixx="0.008637" iyy="0.016397" izz="0.008644" ixy="3e-06" iyz="-0.0" ixz="-0.0"/>
+  </inertial>
+  <visual>
+    <origin xyz="0.205931 0.150121 -0.125" rpy="0 0 0"/>
     <geometry>
       <mesh filename="package://bot5_description/meshes/right_wheel_1.stl" scale="0.001 0.001 0.001"/>
@@ -58,5 +58,5 @@
   </visual>
   <collision>
-    <origin xyz="-0.194069 0.150121 -0.125" rpy="0 0 0"/>
+    <origin xyz="0.205931 0.150121 -0.125" rpy="0 0 0"/>
     <geometry>
       <mesh filename="package://bot5_description/meshes/right_wheel_1.stl" scale="0.001 0.001 0.001"/>
@@ -66,10 +66,10 @@
 <link name="caster_wheel_left_1">
   <inertial>
-    <origin xyz="9.226550963831182e-06 -0.006899932525287894 -4.6891062368895065e-06" rpy="0 0 0"/>
+    <origin xyz="0.20000922655096387 -0.006899932525287894 -4.689106236903384e-06" rpy="0 0 0"/>
     <mass value="0.17837143544148457"/>
     <inertia ixx="0.00012" iyy="0.000221" izz="0.00012" ixy="-0.0" iyz="0.0" ixz="-0.0"/>
   </inertial>
   <visual>
-    <origin xyz="0.21275 -0.105633 -0.049997" rpy="0 0 0"/>
+    <origin xyz="0.61275 -0.105633 -0.049997" rpy="0 0 0"/>
     <geometry>
       <mesh filename="package://bot5_description/meshes/caster_wheel_left_1.stl" scale="0.001 0.001 0.001"/>
@@ -78,5 +78,5 @@
   </visual>
   <collision>
-    <origin xyz="0.21275 -0.105633 -0.049997" rpy="0 0 0"/>
+    <origin xyz="0.61275 -0.105633 -0.049997" rpy="0 0 0"/>
     <geometry>
       <mesh filename="package://bot5_description/meshes/caster_wheel_left_1.stl" scale="0.001 0.001 0.001"/>
@@ -86,10 +86,10 @@
 <link name="caster_body_left_1">
   <inertial>
-    <origin xyz="-0.005218054493926094 -0.00010402054037032815 -0.017359128884011366" rpy="0 0 0"/>
-    <mass value="0.6243519441999044"/>
+    <origin xyz="-0.005218054493926039 -0.00010402054037038366 -0.017359128884011393" rpy="0 0 0"/>
+    <mass value="0.6243519441999045"/>
     <inertia ixx="0.000602" iyy="0.000614" izz="0.00061" ixy="-2e-06" iyz="-4e-06" ixz="-0.000135"/>
   </inertial>
   <visual>
-    <origin xyz="0.178931 -0.099879 -0.127652" rpy="0 0 0"/>
+    <origin xyz="0.378931 -0.099879 -0.127652" rpy="0 0 0"/>
     <geometry>
       <mesh filename="package://bot5_description/meshes/caster_body_left_1.stl" scale="0.001 0.001 0.001"/>
@@ -98,5 +98,5 @@
   </visual>
   <collision>
-    <origin xyz="0.178931 -0.099879 -0.127652" rpy="0 0 0"/>
+    <origin xyz="0.378931 -0.099879 -0.127652" rpy="0 0 0"/>
     <geometry>
       <mesh filename="package://bot5_description/meshes/caster_body_left_1.stl" scale="0.001 0.001 0.001"/>
@@ -106,10 +106,10 @@
 <link name="caster_wheel_right_1">
   <inertial>
-    <origin xyz="9.226550964525071e-06 0.005499857821771828 -4.68910623065838e-06" rpy="0 0 0"/>
+    <origin xyz="0.20000922655096454 0.005499857821771828 -4.68910623065838e-06" rpy="0 0 0"/>
     <mass value="0.1783714354414845"/>
     <inertia ixx="0.00012" iyy="0.000221" izz="0.00012" ixy="0.0" iyz="0.0" ixz="-0.0"/>
   </inertial>
   <visual>
-    <origin xyz="0.21275 0.105875 -0.049997" rpy="0 0 0"/>
+    <origin xyz="0.61275 0.105875 -0.049997" rpy="0 0 0"/>
     <geometry>
       <mesh filename="package://bot5_description/meshes/caster_wheel_right_1.stl" scale="0.001 0.001 0.001"/>
@@ -118,5 +118,5 @@
   </visual>
   <collision>
-    <origin xyz="0.21275 0.105875 -0.049997" rpy="0 0 0"/>
+    <origin xyz="0.61275 0.105875 -0.049997" rpy="0 0 0"/>
     <geometry>
       <mesh filename="package://bot5_description/meshes/caster_wheel_right_1.stl" scale="0.001 0.001 0.001"/>
@@ -126,10 +126,10 @@
 <link name="caster_body_right_1">
   <inertial>
-    <origin xyz="-0.005218047430279288 0.00010393520480088403 -0.017359129924634092" rpy="0 0 0"/>
+    <origin xyz="-0.005218047430279149 0.00010393520480091178 -0.017359129924634106" rpy="0 0 0"/>
     <mass value="0.6243516912268836"/>
     <inertia ixx="0.000602" iyy="0.000614" izz="0.00061" ixy="2e-06" iyz="4e-06" ixz="-0.000135"/>
   </inertial>
   <visual>
-    <origin xyz="0.178931 0.100121 -0.127652" rpy="0 0 0"/>
+    <origin xyz="0.378931 0.100121 -0.127652" rpy="0 0 0"/>
     <geometry>
       <mesh filename="package://bot5_description/meshes/caster_body_right_1.stl" scale="0.001 0.001 0.001"/>
@@ -138,5 +138,5 @@
   </visual>
   <collision>
-    <origin xyz="0.178931 0.100121 -0.127652" rpy="0 0 0"/>
+    <origin xyz="0.378931 0.100121 -0.127652" rpy="0 0 0"/>
     <geometry>
       <mesh filename="package://bot5_description/meshes/caster_body_right_1.stl" scale="0.001 0.001 0.001"/>
@@ -146,10 +146,10 @@
 <link name="realsense_1">
   <inertial>
-    <origin xyz="0.0020983132889169642 0.0011644524543959174 0.01243779695699343" rpy="0 0 0"/>
+    <origin xyz="0.002098313288916971 0.0011644524543959218 0.01243779695699343" rpy="0 0 0"/>
     <mass value="0.09533442052024742"/>
     <inertia ixx="5.9e-05" iyy="9e-06" izz="6e-05" ixy="1e-06" iyz="-0.0" ixz="-0.0"/>
   </inertial>
   <visual>
-    <origin xyz="-0.235069 0.000121 -0.223" rpy="0 0 0"/>
+    <origin xyz="-0.035069 0.000121 -0.223" rpy="0 0 0"/>
     <geometry>
       <mesh filename="package://bot5_description/meshes/realsense_1.stl" scale="0.001 0.001 0.001"/>
@@ -158,5 +158,5 @@
   </visual>
   <collision>
-    <origin xyz="-0.235069 0.000121 -0.223" rpy="0 0 0"/>
+    <origin xyz="-0.035069 0.000121 -0.223" rpy="0 0 0"/>
     <geometry>
       <mesh filename="package://bot5_description/meshes/realsense_1.stl" scale="0.001 0.001 0.001"/>
@@ -166,10 +166,10 @@
 <link name="lidar_1">
   <inertial>
-    <origin xyz="0.000109144073093842 -1.1037922008850449e-05 0.015279585004613405" rpy="0 0 0"/>
+    <origin xyz="0.0001091440730938394 -1.1037922008845516e-05 0.015279585004613405" rpy="0 0 0"/>
     <mass value="0.3162775249943875"/>
     <inertia ixx="6e-05" iyy="6e-05" izz="6.5e-05" ixy="1e-06" iyz="-0.0" ixz="0.0"/>
   </inertial>
   <visual>
-    <origin xyz="-0.195191 0.000121 -0.277" rpy="0 0 0"/>
+    <origin xyz="0.004809 0.000121 -0.277" rpy="0 0 0"/>
     <geometry>
       <mesh filename="package://bot5_description/meshes/lidar_1.stl" scale="0.001 0.001 0.001"/>
@@ -178,5 +178,5 @@
   </visual>
   <collision>
-    <origin xyz="-0.195191 0.000121 -0.277" rpy="0 0 0"/>
+    <origin xyz="0.004809 0.000121 -0.277" rpy="0 0 0"/>
     <geometry>
       <mesh filename="package://bot5_description/meshes/lidar_1.stl" scale="0.001 0.001 0.001"/>
@@ -185,5 +185,5 @@
 </link>
 <joint name="Rev2" type="continuous">
-  <origin xyz="0.194069 0.149879 0.125" rpy="0 0 0"/>
+  <origin xyz="-0.205931 0.149879 0.125" rpy="0 0 0"/>
   <parent link="base_link"/>
   <child link="left_wheel_1"/>
@@ -191,5 +191,5 @@
 </joint>
 <joint name="Rev3" type="continuous">
-  <origin xyz="0.194069 -0.150121 0.125" rpy="0 0 0"/>
+  <origin xyz="-0.205931 -0.150121 0.125" rpy="0 0 0"/>
   <parent link="base_link"/>
   <child link="right_wheel_1"/>
@@ -197,5 +197,5 @@
 </joint>
 <joint name="Rev4" type="continuous">
-  <origin xyz="-0.033819 0.005754 -0.077655" rpy="0 0 0"/>
+  <origin xyz="-0.233819 0.005754 -0.077655" rpy="0 0 0"/>
   <parent link="caster_body_left_1"/>
   <child link="caster_wheel_left_1"/>
@@ -203,5 +203,5 @@
 </joint>
 <joint name="Rev5" type="continuous">
-  <origin xyz="-0.178931 0.099879 0.127652" rpy="0 0 0"/>
+  <origin xyz="-0.378931 0.099879 0.127652" rpy="0 0 0"/>
   <parent link="base_link"/>
   <child link="caster_body_left_1"/>
@@ -209,5 +209,5 @@
 </joint>
 <joint name="Rev6" type="continuous">
-  <origin xyz="-0.033819 -0.005754 -0.077655" rpy="0 0 0"/>
+  <origin xyz="-0.233819 -0.005754 -0.077655" rpy="0 0 0"/>
   <parent link="caster_body_right_1"/>
   <child link="caster_wheel_right_1"/>
@@ -215,5 +215,5 @@
 </joint>
 <joint name="Rev7" type="continuous">
-  <origin xyz="-0.178931 -0.100121 0.127652" rpy="0 0 0"/>
+  <origin xyz="-0.378931 -0.100121 0.127652" rpy="0 0 0"/>
   <parent link="base_link"/>
   <child link="caster_body_right_1"/>
@@ -221,10 +221,10 @@
 </joint>
 <joint name="Rigid8" type="fixed">
-  <origin xyz="0.235069 -0.000121 0.223" rpy="0 0 0"/>
+  <origin xyz="0.035069 -0.000121 0.223" rpy="0 0 0"/>
   <parent link="base_link"/>
   <child link="realsense_1"/>
 </joint>
 <joint name="Rigid9" type="fixed">
-  <origin xyz="0.195191 -0.000121 0.277" rpy="0 0 0"/>
+  <origin xyz="-0.004809 -0.000121 0.277" rpy="0 0 0"/>
   <parent link="base_link"/>
   <child link="lidar_1"/>

Commit message: Wheel parameters fixed
to match HB controller odometry.

Dummy link added

File: urdf/bot5.xacro (robot description, xacro)
@@ -4,4 +4,5 @@
 <xacro:include filename="$(find bot5_description)/urdf/bot5.trans" />
 <xacro:include filename="$(find bot5_description)/urdf/bot5.gazebo" />
+<link name="dummy"/>
 <link name="base_link">
   <inertial>
@@ -24,5 +25,9 @@
   </collision>
 </link>
-<link name="left_wheel_1">
+<joint name="dummy_joint" type="fixed">
+ <parent link="dummy"/>
+ <child link="base_footprint"/>
+</joint>
+<link name="left_wheel">
   <inertial>
     <origin xyz="0.20004860168806374 0.03873115898033333 -4.449218771185315e-14" rpy="0 0 0"/>
@@ -44,5 +49,5 @@
   </collision>
 </link>
-<link name="right_wheel_1">
+<link name="right_wheel">
   <inertial>
     <origin xyz="0.20004860168807084 -0.03873122504117252 -4.4103609653234344e-14" rpy="0 0 0"/>
@@ -184,14 +189,14 @@
   </collision>
 </link>
-<joint name="Rev2" type="continuous">
+<joint name="left_wheel" type="continuous">
   <origin xyz="-0.205931 0.149879 0.125" rpy="0 0 0"/>
   <parent link="base_link"/>
-  <child link="left_wheel_1"/>
+  <child link="left_wheel"/>
   <axis xyz="-0.0 1.0 -0.0"/>
 </joint>
-<joint name="Rev3" type="continuous">
+<joint name="right_wheel" type="continuous">
   <origin xyz="-0.205931 -0.150121 0.125" rpy="0 0 0"/>
   <parent link="base_link"/>
-  <child link="right_wheel_1"/>
+  <child link="right_wheel"/>
   <axis xyz="-0.0 1.0 -0.0"/>
 </joint>

Commit message: Add files via upload

File: urdf/bot5.xacro (robot description, xacro)
@@ -4,5 +4,4 @@
 <xacro:include filename="$(find bot5_description)/urdf/bot5.trans" />
 <xacro:include filename="$(find bot5_description)/urdf/bot5.gazebo" />
-<link name="dummy"/>
 <link name="base_link">
   <inertial>
@@ -25,9 +24,5 @@
   </collision>
 </link>
-<joint name="dummy_joint" type="fixed">
- <parent link="dummy"/>
- <child link="base_footprint"/>
-</joint>
-<link name="left_wheel">
+<link name="left_wheel_1">
   <inertial>
     <origin xyz="0.20004860168806374 0.03873115898033333 -4.449218771185315e-14" rpy="0 0 0"/>
@@ -49,5 +44,5 @@
   </collision>
 </link>
-<link name="right_wheel">
+<link name="right_wheel_1">
   <inertial>
     <origin xyz="0.20004860168807084 -0.03873122504117252 -4.4103609653234344e-14" rpy="0 0 0"/>
@@ -189,14 +184,14 @@
   </collision>
 </link>
-<joint name="left_wheel" type="continuous">
+<joint name="Rev2" type="continuous">
   <origin xyz="-0.205931 0.149879 0.125" rpy="0 0 0"/>
   <parent link="base_link"/>
-  <child link="left_wheel"/>
+  <child link="left_wheel_1"/>
   <axis xyz="-0.0 1.0 -0.0"/>
 </joint>
-<joint name="right_wheel" type="continuous">
+<joint name="Rev3" type="continuous">
   <origin xyz="-0.205931 -0.150121 0.125" rpy="0 0 0"/>
   <parent link="base_link"/>
-  <child link="right_wheel"/>
+  <child link="right_wheel_1"/>
   <axis xyz="-0.0 1.0 -0.0"/>
 </joint>

Commit message: Update bot5.xacro

File: urdf/bot5.xacro (robot description, xacro)
@@ -4,4 +4,5 @@
 <xacro:include filename="$(find bot5_description)/urdf/bot5.trans" />
 <xacro:include filename="$(find bot5_description)/urdf/bot5.gazebo" />
+<link name="dummy"/>
 <link name="base_link">
   <inertial>
@@ -24,5 +25,9 @@
   </collision>
 </link>
-<link name="left_wheel_1">
+    <joint name="dummy_joint" type="fixed">
+     <parent link="dummy"/>
+     <child link="base_link"/>
+     </joint>
+<link name="left_wheel">
   <inertial>
     <origin xyz="0.20004860168806374 0.03873115898033333 -4.449218771185315e-14" rpy="0 0 0"/>
@@ -44,5 +49,5 @@
   </collision>
 </link>
-<link name="right_wheel_1">
+<link name="right_wheel">
   <inertial>
     <origin xyz="0.20004860168807084 -0.03873122504117252 -4.4103609653234344e-14" rpy="0 0 0"/>

Commit message: Update bot5.xacro

File: urdf/bot5.xacro (robot description, xacro)
@@ -24,5 +24,5 @@
   </collision>
 </link>
-<link name="left_wheel_1">
+<link name="left_wheel">
   <inertial>
     <origin xyz="4.860168806373845e-05 0.03933115898033335 -4.4422798772814076e-14" rpy="0 0 0"/>
@@ -44,5 +44,5 @@
   </collision>
 </link>
-<link name="right_wheel_1">
+<link name="right_wheel">
   <inertial>
     <origin xyz="4.860168807075394e-05 -0.039331225041172535 -4.4075854077618715e-14" rpy="0 0 0"/>
@@ -144,5 +144,5 @@
   </collision>
 </link>
-<link name="realsense_1">
+<link name="realsense">
   <inertial>
     <origin xyz="0.006048313146213111 0.0011644524543970541 0.012437796956994596" rpy="0 0 0"/>
@@ -164,5 +164,5 @@
   </collision>
 </link>
-<link name="imu_1">
+<link name="imu">
   <inertial>
     <origin xyz="1.9553994023285837e-07 -3.303041936634414e-08 0.001000001415556534" rpy="0 0 0"/>
@@ -184,5 +184,5 @@
   </collision>
 </link>
-<link name="lidar_1">
+<link name="lidar">
   <inertial>
     <origin xyz="0.0001091440734231734 -1.1037922009016115e-05 0.01727958500461163" rpy="0 0 0"/>
@@ -207,5 +207,5 @@
   <origin xyz="6.9e-05 0.149879 0.125" rpy="0 0 0"/>
   <parent link="base_link"/>
-  <child link="left_wheel_1"/>
+  <child link="left_wheel"/>
   <axis xyz="-0.0 1.0 -0.0"/>
 </joint>
@@ -213,5 +213,5 @@
   <origin xyz="6.9e-05 -0.150121 0.125" rpy="0 0 0"/>
   <parent link="base_link"/>
-  <child link="right_wheel_1"/>
+  <child link="right_wheel"/>
   <axis xyz="-0.0 1.0 -0.0"/>
 </joint>
@@ -243,15 +243,15 @@
   <origin xyz="0.034069 -0.000121 0.223" rpy="0 0 0"/>
   <parent link="base_link"/>
-  <child link="realsense_1"/>
-</joint>
-<joint name="Rigid8" type="fixed">
+  <child link="realsense"/>
+</joint>
+<joint name="imu" type="fixed">
   <origin xyz="0.041069 -0.000121 0.223" rpy="0 0 0"/>
   <parent link="base_link"/>
-  <child link="imu_1"/>
-</joint>
-<joint name="Rigid9" type="fixed">
+  <child link="imu"/>
+</joint>
+<joint name="lidar" type="fixed">
   <origin xyz="0.001191 -0.000121 0.277" rpy="0 0 0"/>
   <parent link="base_link"/>
-  <child link="lidar_1"/>
+  <child link="lidar"/>
 </joint>
 </robot>
