Commit message: Add files via upload

File: urdf/bot5.xacro (robot description, xacro)
@@ -1,7 +1,7 @@
 <?xml version="1.0" ?>
 <robot name="bot5" xmlns:xacro="http://www.ros.org/wiki/xacro">
-<xacro:include filename="$(find bot5_description)/urdf/materials.xacro" />
-<xacro:include filename="$(find bot5_description)/urdf/bot5.trans" />
-<xacro:include filename="$(find bot5_description)/urdf/bot5.gazebo" />
+<xacro:include filename="$(find bot5)/urdf/materials.xacro" />
+<xacro:include filename="$(find bot5)/urdf/bot5.trans" />
+<xacro:include filename="$(find bot5)/urdf/bot5.gazebo" />
 <link name="base_link">
   <inertial>
@@ -13,5 +13,5 @@
     <origin xyz="0 0 0" rpy="0 0 0"/>
     <geometry>
-      <mesh filename="package://bot5_description/meshes/base_link.stl" scale="0.001 0.001 0.001"/>
+      <mesh filename="package://bot5/meshes/base_link.stl" scale="0.001 0.001 0.001"/>
     </geometry>
     <material name="silver"/>
@@ -20,5 +20,5 @@
     <origin xyz="0 0 0" rpy="0 0 0"/>
     <geometry>
-      <mesh filename="package://bot5_description/meshes/base_link.stl" scale="0.001 0.001 0.001"/>
+      <mesh filename="package://bot5/meshes/base_link.stl" scale="0.001 0.001 0.001"/>
     </geometry>
   </collision>
@@ -33,5 +33,5 @@
     <origin xyz="-6.9e-05 -0.149879 -0.125" rpy="0 0 0"/>
     <geometry>
-      <mesh filename="package://bot5_description/meshes/left_wheel_1.stl" scale="0.001 0.001 0.001"/>
+      <mesh filename="package://bot5/meshes/left_wheel_1.stl" scale="0.001 0.001 0.001"/>
     </geometry>
     <material name="silver"/>
@@ -40,5 +40,5 @@
     <origin xyz="-6.9e-05 -0.149879 -0.125" rpy="0 0 0"/>
     <geometry>
-      <mesh filename="package://bot5_description/meshes/left_wheel_1.stl" scale="0.001 0.001 0.001"/>
+      <mesh filename="package://bot5/meshes/left_wheel_1.stl" scale="0.001 0.001 0.001"/>
     </geometry>
   </collision>
@@ -53,5 +53,5 @@
     <origin xyz="-6.9e-05 0.150121 -0.125" rpy="0 0 0"/>
     <geometry>
-      <mesh filename="package://bot5_description/meshes/right_wheel_1.stl" scale="0.001 0.001 0.001"/>
+      <mesh filename="package://bot5/meshes/right_wheel_1.stl" scale="0.001 0.001 0.001"/>
     </geometry>
     <material name="silver"/>
@@ -60,5 +60,5 @@
     <origin xyz="-6.9e-05 0.150121 -0.125" rpy="0 0 0"/>
     <geometry>
-      <mesh filename="package://bot5_description/meshes/right_wheel_1.stl" scale="0.001 0.001 0.001"/>
+      <mesh filename="package://bot5/meshes/right_wheel_1.stl" scale="0.001 0.001 0.001"/>
     </geometry>
   </collision>
@@ -73,5 +73,5 @@
     <origin xyz="0.40775 -0.090375 -0.049995" rpy="0 0 0"/>
     <geometry>
-      <mesh filename="package://bot5_description/meshes/caster_wheel_left_1.stl" scale="0.001 0.001 0.001"/>
+      <mesh filename="package://bot5/meshes/caster_wheel_left_1.stl" scale="0.001 0.001 0.001"/>
     </geometry>
     <material name="silver"/>
@@ -80,5 +80,5 @@
     <origin xyz="0.40775 -0.090375 -0.049995" rpy="0 0 0"/>
     <geometry>
-      <mesh filename="package://bot5_description/meshes/caster_wheel_left_1.stl" scale="0.001 0.001 0.001"/>
+      <mesh filename="package://bot5/meshes/caster_wheel_left_1.stl" scale="0.001 0.001 0.001"/>
     </geometry>
   </collision>
@@ -93,5 +93,5 @@
     <origin xyz="0.40775 0.105875 -0.049995" rpy="0 0 0"/>
     <geometry>
-      <mesh filename="package://bot5_description/meshes/caster_wheel_right_1.stl" scale="0.001 0.001 0.001"/>
+      <mesh filename="package://bot5/meshes/caster_wheel_right_1.stl" scale="0.001 0.001 0.001"/>
     </geometry>
     <material name="silver"/>
@@ -100,5 +100,5 @@
     <origin xyz="0.40775 0.105875 -0.049995" rpy="0 0 0"/>
     <geometry>
-      <mesh filename="package://bot5_description/meshes/caster_wheel_right_1.stl" scale="0.001 0.001 0.001"/>
+      <mesh filename="package://bot5/meshes/caster_wheel_right_1.stl" scale="0.001 0.001 0.001"/>
     </geometry>
   </collision>
@@ -113,5 +113,5 @@
     <origin xyz="0.372931 -0.099879 -0.127652" rpy="0 0 0"/>
     <geometry>
-      <mesh filename="package://bot5_description/meshes/caster_body_left_1.stl" scale="0.001 0.001 0.001"/>
+      <mesh filename="package://bot5/meshes/caster_body_left_1.stl" scale="0.001 0.001 0.001"/>
     </geometry>
     <material name="silver"/>
@@ -120,5 +120,5 @@
     <origin xyz="0.372931 -0.099879 -0.127652" rpy="0 0 0"/>
     <geometry>
-      <mesh filename="package://bot5_description/meshes/caster_body_left_1.stl" scale="0.001 0.001 0.001"/>
+      <mesh filename="package://bot5/meshes/caster_body_left_1.stl" scale="0.001 0.001 0.001"/>
     </geometry>
   </collision>
@@ -133,5 +133,5 @@
     <origin xyz="0.372931 0.100121 -0.127652" rpy="0 0 0"/>
     <geometry>
-      <mesh filename="package://bot5_description/meshes/caster_body_right_1.stl" scale="0.001 0.001 0.001"/>
+      <mesh filename="package://bot5/meshes/caster_body_right_1.stl" scale="0.001 0.001 0.001"/>
     </geometry>
     <material name="silver"/>
@@ -140,9 +140,9 @@
     <origin xyz="0.372931 0.100121 -0.127652" rpy="0 0 0"/>
     <geometry>
-      <mesh filename="package://bot5_description/meshes/caster_body_right_1.stl" scale="0.001 0.001 0.001"/>
-    </geometry>
-  </collision>
-</link>
-<link name="realsense">
+      <mesh filename="package://bot5/meshes/caster_body_right_1.stl" scale="0.001 0.001 0.001"/>
+    </geometry>
+  </collision>
+</link>
+<link name="camera_link">
   <inertial>
     <origin xyz="0.006048313146213111 0.0011644524543970541 0.012437796956994596" rpy="0 0 0"/>
@@ -153,5 +153,5 @@
     <origin xyz="-0.034069 0.000121 -0.223" rpy="0 0 0"/>
     <geometry>
-      <mesh filename="package://bot5_description/meshes/realsense_1.stl" scale="0.001 0.001 0.001"/>
+      <mesh filename="package://bot5/meshes/realsense_1.stl" scale="0.001 0.001 0.001"/>
     </geometry>
     <material name="silver"/>
@@ -160,5 +160,5 @@
     <origin xyz="-0.034069 0.000121 -0.223" rpy="0 0 0"/>
     <geometry>
-      <mesh filename="package://bot5_description/meshes/realsense_1.stl" scale="0.001 0.001 0.001"/>
+      <mesh filename="package://bot5/meshes/realsense_1.stl" scale="0.001 0.001 0.001"/>
     </geometry>
   </collision>
@@ -173,5 +173,5 @@
     <origin xyz="-0.041069 0.000121 -0.223" rpy="0 0 0"/>
     <geometry>
-      <mesh filename="package://bot5_description/meshes/imu_1.stl" scale="0.001 0.001 0.001"/>
+      <mesh filename="package://bot5/meshes/imu_1.stl" scale="0.001 0.001 0.001"/>
     </geometry>
     <material name="silver"/>
@@ -180,5 +180,5 @@
     <origin xyz="-0.041069 0.000121 -0.223" rpy="0 0 0"/>
     <geometry>
-      <mesh filename="package://bot5_description/meshes/imu_1.stl" scale="0.001 0.001 0.001"/>
+      <mesh filename="package://bot5/meshes/imu_1.stl" scale="0.001 0.001 0.001"/>
     </geometry>
   </collision>
@@ -193,5 +193,5 @@
     <origin xyz="-0.001191 0.000121 -0.277" rpy="0 0 0"/>
     <geometry>
-      <mesh filename="package://bot5_description/meshes/lidar_1.stl" scale="0.001 0.001 0.001"/>
+      <mesh filename="package://bot5/meshes/lidar_1.stl" scale="0.001 0.001 0.001"/>
     </geometry>
     <material name="silver"/>
@@ -200,5 +200,5 @@
     <origin xyz="-0.001191 0.000121 -0.277" rpy="0 0 0"/>
     <geometry>
-      <mesh filename="package://bot5_description/meshes/lidar_1.stl" scale="0.001 0.001 0.001"/>
+      <mesh filename="package://bot5/meshes/lidar_1.stl" scale="0.001 0.001 0.001"/>
     </geometry>
   </collision>
@@ -240,8 +240,8 @@
   <axis xyz="0.0 0.0 1.0"/>
 </joint>
-<joint name="realsense" type="fixed">
+<joint name="camera_joint" type="fixed">
   <origin xyz="0.034069 -0.000121 0.223" rpy="0 0 0"/>
   <parent link="base_link"/>
-  <child link="realsense"/>
+  <child link="camera_link"/>
 </joint>
 <joint name="imu" type="fixed">
